Commit message: Imported upstream version '0.2.4' of 'upstream'

File: spur_description/urdf/spur.urdf.xacro (robot description, xacro)
@@ -13,5 +13,5 @@
   <property name="wheel_radius" value="0.05" />
   <property name="wheel_width" value="0.02" />
-  <property name="base_width" value="0.430" />
+  <property name="base_width" value="0.30" />
   <property name="base_height" value="0.030" />
   <property name="caster_offset_x" value="0.15" />
@@ -307,5 +307,5 @@
     </inertial>
     <visual>
-      <origin xyz="0 0 0" rpy="3.14 0 0"/>
+      <origin xyz="0 0 0" rpy="0 0 0"/>
       <geometry>
       <!-- <cylinder length="${hokuyo_length}" radius="${hokuyo_radius}" /> -->
@@ -321,5 +321,5 @@
   </link>
   <joint name="laser_to_base" type="fixed">
-    <origin xyz="${caster_offset_x} 0 -0.05" rpy="0 0 0" />
+    <origin xyz="${caster_offset_x} 0 -0.05" rpy="3.14 0 0" />
     <parent link="base_link" />
     <child link="hokuyo_sensor_link"/>
