Commit message: Imported upstream version '0.2.6' of 'upstream'

File: spur_description/urdf/spur.gazebo.xacro (robot description, xacro)
@@ -12,23 +12,42 @@
       <robotNamespace>/${ns}</robotNamespace>
     </plugin>
+    <plugin name="ground_truth" filename="libgazebo_ros_p3d.so">
+      <frameName>map</frameName>
+      <bodyName>base_footprint</bodyName>
+      <topicName>base_pose_ground_truth</topicName>
+      <updateRate>30.0</updateRate>
+    </plugin>
   </gazebo>
-  <xacro:macro name="gazebo_link" params="name color">
+  <xacro:macro name="gazebo_tire_link" params="name color">
     <gazebo reference="${name}">
       <material>Gazebo/${color}</material>
-      <mu1 value="1.0" />
-      <mu2 value="1.0" />
-      <kp value="10000000.0" />
-      <kd value="1.0" />
+      <kp>100000.0</kp>
+      <kd>10.0</kd>
+      <mu1>1</mu1>
+      <mu2>1</mu2>
+      <fdir1>1 0 0</fdir1>
+      <minDepth>0.003</minDepth>
+      <maxVel>1.0</maxVel>
     </gazebo>
   </xacro:macro>
-  <xacro:macro name="simple_transmission" params="name" >
+  <xacro:macro name="gazebo_base_link" params="name color">
+    <gazebo reference="${name}">
+      <material>Gazebo/${color}</material>
+    </gazebo>
+  </xacro:macro>
+  <xacro:macro name="gazebo_arm_link" params="name color">
+    <gazebo reference="${name}">
+      <material>Gazebo/${color}</material>
+    </gazebo>
+  </xacro:macro>
+  <xacro:macro name="simple_transmission" params="name interface" >
     <transmission name="${name}_trans">
       <type>transmission_interface/SimpleTransmission</type>
       <joint name="${name}">
-        <hardwareInterface>EffortJointInterface</hardwareInterface>
+        <hardwareInterface>${interface}</hardwareInterface>
       </joint>
       <actuator name="${name}_motor">
-        <hardwareInterface>EffortJointInterface</hardwareInterface>
-        <mechanicalReduction>1</mechanicalReduction>
+        <mechanicalReduction>10</mechanicalReduction>
+        <hardwareInterface>${interface}</hardwareInterface>
       </actuator>
     </transmission>
@@ -44,17 +63,18 @@
           <scan>
             <horizontal>
-              <samples>720</samples>
+              <!-- The URG-04LX-UG01  has  683 steps with 0.35139 Degree resolution -->
+              <samples>683</samples>
               <resolution>1</resolution>
-              <min_angle>-1.570796</min_angle>
-              <max_angle>1.570796</max_angle>
+              <min_angle>-2.0944</min_angle> <!-- 120 Degree -->
+              <max_angle>2.0944</max_angle>
             </horizontal>
           </scan>
           <range>
-            <min>0.1</min>
-            <max>4.0</max>
+            <min>0.06</min> <!-- 0.06 from URG-04 specification -->
+            <max>10.0</max>
             <resolution>0.01</resolution>
           </range>
           <noise>
-            <type>Gaussian</type>
+            <type>gaussian</type>
             <mean>0.0</mean>
             <stddev>0.01</stddev>
